File: schematics/Orion68/_autosave-orion68cpu2.kicad_sch (KiCad schematic)
At the start: 48 parts, among them J1 clock, Q1 2N3904, Q2 2N3904, Q3 2N3904, SW2 reset, U0 74LS393, U10 SST39SF010, U11 MC68000FN, U2 74LS541, U3 74LS541, U4 74LS541, U5 74LS245, U6 74LS245, U7 74LS541, U8 74LS148, U9 SST39SF010

Commit message: updating
Parts:
- removed R7, R8: 470R, symbol Device:R
Connections:
- net +5V: now also U10.31 (PGM), U9.31 (PGM)
- net GND: now also D3.1 (K), D4.1 (K)
- net /BERR: now also U11.24 (~{BERR})
- net /halt: now also D3.2 (A)
- net /reset: now also D4.2 (A)
- net at U9.30 (NC): no longer U10.30 (NC)
Other:
- moved on the sheet: D3, D4
