File: schematics/Orion68/orion68cpu.kicad_sch (KiCad schematic)
At the start: 18 parts, among them J2 RTC_NVEM, SW1 reset, U1 MC68000P, U2.1 ATmega8-16P, U2.2 ATmega8-16P, U3 74LS05, U4 74HC14, Y1 16MHZ, Y1.1 16MHZ

Commit message: Updating cpu
Parts:
- renumbered D2 to D1, D1 to D2, J1 to J3, R5 to R1, R4 to R2, R2 to R4, R1 to R5, U3 to U1, U4 to U2, U1 to U3
