File: schematics/Orion68/orion68cpu2.kicad_sch (KiCad schematic)
At the start: 54 parts, among them J1 Euro96pin, J2 clock, Q1 2N3904, Q2 2N3904, Q3 2N3904, SW2 sw_reset, U0 MC68000FN, U1 74LS245, U10 SST39SF010, U11 74HC74, U12 74LS393, U2 74LS245, U3 74LS541, U4 74LS541, U5 74LS541, U6 74LS541, U7 74LS148, U8 GAL16V8, U9 SST39SF010

Commit message: Schematics update
Parts:
- removed J2: clock, Connector_PinHeader_2.54mm:PinHeader_2x04_P2.54mm_Vertical, symbol Connector_Generic:Conn_02x04_Counter_Clockwise
- added C_U13: 100nF, Capacitor_THT:C_Disc_D4.3mm_W1.9mm_P5.00mm, symbol Device:C
- added J2: clock, symbol Connector_Generic:Conn_02x05_Counter_Clockwise
- added J3: clock1, symbol Connector_Generic:Conn_02x04_Counter_Clockwise
- added R16, R4, R5: 270R, Resistor_THT:R_Axial_DIN0204_L3.6mm_D1.6mm_P5.08mm_Horizontal, symbol Device:R
- added R3: 4k7, Resistor_THT:R_Axial_DIN0204_L3.6mm_D1.6mm_P5.08mm_Horizontal, symbol Device:R
- added U13: PAL20RS10, Package_DIP:DIP-24_W7.62mm, symbol Logic_Programmable:PAL20RS10
Connections:
- net PWR_GOOD_IN is gone; now on net PWR_GOOD: J1.88
- net +5V: now also C_U13.1, R16.2, R3.1, R5.2, U13.24 (VCC)
- net 16MHZ: now also J2.1 (Pin_1)
- net 1MHZ: now also U12.13 (CP), J2.9 (Pin_9)
- net 2MHZ: now also J2.7 (Pin_7)
- net 4MHZ: now also J2.5 (Pin_5)
- net 8MHZ: now also J2.3 (Pin_3)
- net A1: now also U13.10 (I8)
- net A2: now also U13.11 (I9)
- net A3: now also U13.13 (~{OE})
- net BA23: now also J1.54
- net BOOTIN: now also J1.87, R4.2; no longer D4.2 (A)
- net B/cpurd: now also J1.45
- net CPU_CLK: now also J2.10 (Pin_10), J2.2 (Pin_2), J2.4 (Pin_4), J2.6 (Pin_6), J2.8 (Pin_8)
- net GND: now also U8.11 (I10/~{OE}), C_U13.2, U13.12 (GND); no longer D2.1 (K), D3.1 (K), U12.13 (CP)
- net IRQ2: now also J1.48; no longer J1.49
- net IRQ3: now also J1.49; no longer J1.50
- net IRQ4: now also J1.50, RN1.9 (R8); no longer J1.54, RN1.6 (R5)
- net IRQ5: now also RN1.8 (R7); no longer RN1.7 (R6)
- net IRQ6: now also RN1.7 (R6); no longer RN1.8 (R7)
- net IRQ7: now also RN1.6 (R5); no longer RN1.9 (R8)
- net cpu_fc0: now also U13.6 (I4)
- net cpu_fc1: now also U13.7 (I5)
- net cpu_fc2: now also U13.8 (I6)
- net /HALT: now also D2.1 (K); no longer D2.2 (A)
- net /IO_CS: now also J1.85
- net /RESET: now also D3.1 (K); no longer D3.2 (A)
- net /cpu_ipl0: now also U13.22 (O1); no longer U7.9 (S0)
- net /cpu_ipl2: now also U13.20 (O3); no longer U7.6 (S2)
- net /cpurd: no longer J1.45
- net 250khz: now reaches U12.10 (Q1)
- net 250khz: now also J3.2 (Pin_2)
- net 500khz: now reaches U12.11 (Q0)
- net 500khz: now also J3.1 (Pin_1)
- net 62,5khz: now reaches U12.8 (Q3)
- net 62,5khz: now also J3.4 (Pin_4)
- net 125khz: now reaches U12.9 (Q2)
- net 125khz: now also J3.3 (Pin_3)
- net TICK_IN: now reaches J1.86
- net TICK_IN: now also R3.2, U13.1 (CLK)
- net GS_148: now reaches U7.14 (GS)
- net GS_148: now also U13.5 (I3)
- net IRQ1: no longer names the net of RN1.3 (R2), U7.11 (I1)
- net IRQ1: no longer J1.48
- net /cpu_ipl1: no longer names the net of U0.26 (~{IPL1})
- net /cpu_ipl1: now also U13.21 (O2); no longer U7.7 (S1)
- net /cpurw renamed B/cpurw
- new net: J3.5 (Pin_5), J3.6 (Pin_6), J3.7 (Pin_7), J3.8 (Pin_8)
- new net: D4.2 (A), R4.1
- new net: D3.2 (A), R5.1
- new net: D2.2 (A), R16.1
- new net A0_148: U13.2 (I0), U7.9 (S0)
- new net A1_148: U13.3 (I1), U7.7 (S1)
- new net A2_148: U13.4 (I2), U7.6 (S2)
- new net AS: U13.9 (I7)
- new net IRQ_S: U13.23 (O0)
- no-connect marks 4 -> 3
Other:
- moved on the sheet: C2, D1, D2, D3, D4, J1, Q1, Q2, R10, R2, R6, R7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
