File: schematics/Orion68/Orion68.kicad_pcb (KiCad board)
At the start: 2 copper layers, 55 parts, among them J1 Euro96pin, J2 clock, Q1 2N3904, Q2 2N3904, Q3 2N3904, SW2 sw_reset, U0 MC68000FN, U1 74LS245, U10 SST39SF010, U11 74HC74, U12 74LS393, U2 74LS245, U3 74LS541, U4 74LS541, U5 74LS541, U6 74LS541, U7 74LS148, U8 GAL16V8, U9 SST39SF010

Commit message: Schematics update
Parts:
- removed J2: clock, Connector_PinHeader_2.54mm:PinHeader_2x04_P2.54mm_Vertical
- added C_U13: 100nF, Capacitor_THT:C_Disc_D4.3mm_W1.9mm_P5.00mm, F.Cu at (92.2, 116.7)
- added R16: 270R, Resistor_THT:R_Axial_DIN0204_L3.6mm_D1.6mm_P5.08mm_Horizontal, F.Cu at (61.7, 79.1)
- added R3: 4k7, Resistor_THT:R_Axial_DIN0204_L3.6mm_D1.6mm_P5.08mm_Horizontal, F.Cu at (92.1, 113.6)
- added R4: 270R, Resistor_THT:R_Axial_DIN0204_L3.6mm_D1.6mm_P5.08mm_Horizontal, F.Cu at (61.7, 94.3)
- added R5: 270R, Resistor_THT:R_Axial_DIN0204_L3.6mm_D1.6mm_P5.08mm_Horizontal, F.Cu at (61.8, 86.5)
- added U13: PAL20RS10, Package_DIP:DIP-24_W7.62mm, F.Cu at (84.7, 119.8)
- moved R2 114.8 mm to (83.8, 80.5), turned to 180 degrees
- moved RN1 27.2 mm to (112.6, 147.3), turned to 90 degrees
- moved Q3 16.5 mm to (84.9, 56.4), turned to 180 degrees
- moved D2 14.8 mm to (53.6, 79.1)
- moved D3 14.8 mm to (53.6, 86.6)
- moved D4 14.8 mm to (53.6, 94.5)
- moved C2 9.33 mm to (73.0, 73.1)
- moved D1 9.33 mm to (75.0, 79.4)
- moved Q2 9.33 mm to (87.5, 77.6)
- moved R10 9.33 mm to (78.2, 71.4)
- moved R7 9.33 mm to (82.7, 63.6)
- moved R8 9.33 mm to (83.6, 76.4)
- moved R9 9.33 mm to (78.2, 68.6)
- moved Q1 9.33 mm to (87.1, 62.4)
- moved R6 9.33 mm to (70.7, 79.5)
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Connections:
- D2 pad 1: GND -> /Orion68-CPU-2//HALT
- D2 pad 2: /Orion68-CPU-2//HALT -> Net-(D2-A)
- D3 pad 1: GND -> /Orion68-CPU-2//RESET
- D3 pad 2: /Orion68-CPU-2//RESET -> Net-(D3-A)
- D4 pad 2: /Orion68-CPU-2/BOOT_SIG -> Net-(D4-A)
- J1 pad 48: IRQ1 -> IRQ2
- J1 pad 49: IRQ2 -> IRQ3
- J1 pad 50: IRQ3 -> IRQ4
- J1 pad 54: IRQ4 -> unconnected-(J1-Pad54)
- J1 pad 88: /Orion68-CPU-2/PWR_GOOD_IN -> /Orion68-CPU-2/PWR_GOOD
- RN1 pad 3: IRQ1 -> Net-(RN1-R2)
- RN1 pad 6: IRQ4 -> IRQ7
- RN1 pad 7: IRQ5 -> IRQ6
- RN1 pad 8: IRQ6 -> IRQ5
- RN1 pad 9: IRQ7 -> IRQ4
- U0 pad 26: /Orion68-CPU-2//cpu_ipl1 -> /Orion68-CPU-2/<NO NET>
- U12 pad 10: unconnected-(U12B-Q1-Pad10) -> /Orion68-CPU-2/250khz
- U12 pad 11: unconnected-(U12B-Q0-Pad11) -> /Orion68-CPU-2/500khz
- U12 pad 13: GND -> /Orion68-CPU-2/1MHZ
- U12 pad 8: unconnected-(U12B-Q3-Pad8) -> /Orion68-CPU-2/62,5khz
- U12 pad 9: unconnected-(U12B-Q2-Pad9) -> /Orion68-CPU-2/125khz
- U7 pad 11: IRQ1 -> Net-(RN1-R2)
- U7 pad 14: unconnected-(U7-GS-Pad14) -> /Orion68-CPU-2/GS_148
- U7 pad 6: /Orion68-CPU-2//cpu_ipl2 -> /Orion68-CPU-2/A2_148
- U7 pad 7: /Orion68-CPU-2//cpu_ipl1 -> /Orion68-CPU-2/A1_148
- U7 pad 9: /Orion68-CPU-2//cpu_ipl0 -> /Orion68-CPU-2/A0_148
- U8 pad 11: unconnected-(U8-I10/~{OE}-Pad11) -> GND
- U8 pad 15: /Orion68-CPU-2//RD -> unconnected-(U8-IO5-Pad15)
- U8 pad 7: /Orion68-CPU-2/R/W -> unconnected-(U8-I7-Pad7)

Commit message: Schematics update
Parts:
- removed J0: ~, ConnPdSilva:conn_euro96
Connections:
- J1 pad 43: /Orion68-CPU-2//AS -> /Orion68-CPU-2/B/AS
- J1 pad 45: /Orion68-CPU-2//cpurd -> /Orion68-CPU-2/B/cpurd
- J1 pad 46: /Orion68-CPU-2//cpurw -> /Orion68-CPU-2/B/cpuwr
- J1 pad 54: unconnected-(J1-Pad54) -> /Orion68-CPU-2/BA23
- J1 pad 70: /Orion68-CPU-2//LDS -> /Orion68-CPU-2/B/LDS
- J1 pad 71: /Orion68-CPU-2//UDS -> /Orion68-CPU-2/B/UDS
- J1 pad 85: unconnected-(J1-Pad85) -> /Orion68-CPU-2//IO_CS
- J1 pad 86: unconnected-(J1-Pad86) -> /Orion68-CPU-2/TICK_IN
- J1 pad 87: unconnected-(J1-Pad87) -> /Orion68-CPU-2/BOOTIN

Commit message: Updating
Parts:
- added C300: 10pF, Capacitor_THT:C_Disc_D4.3mm_W1.9mm_P5.00mm, F.Cu at (343.7, 56.5)
- added C_S400: 100uF, Capacitor_THT:CP_Radial_D5.0mm_P2.50mm, F.Cu at (310.8, 244.2)
- added D_S300: LED, Diode_THT:D_T-1_P5.08mm_Horizontal, F.Cu at (249.1, 169.8)
- added J100: Euro96pin, ConnPdSilva:conn_euro96, F.Cu at (159.6, 138.6)
- added J2: clock, Connector_PinHeader_2.54mm:PinHeader_2x05_P2.54mm_Vertical, F.Cu at (73.7, 37.7)
- added J200: Euro96pin, ConnPdSilva:conn_euro96, F.Cu at (375.3, 140.6)
- added J3: clock1, Connector_PinHeader_2.54mm:PinHeader_2x04_P2.54mm_Vertical, F.Cu at (60.7, 37.5)
- added J300: Euro96pin, ConnPdSilva:conn_euro96, F.Cu at (374.1, 23.0)
- added J_S100: DB25_Socket, Connector_PinHeader_2.54mm:PinHeader_2x13_P2.54mm_Vertical, F.Cu at (329.2, 140.8)
- added J_S200: sdcard, Connector_PinSocket_2.54mm:PinSocket_1x06_P2.54mm_Vertical, F.Cu at (319.6, 222.9)
- added J_S201: RTC, Connector_PinSocket_2.54mm:PinSocket_1x06_P2.54mm_Vertical, F.Cu at (311.3, 168.6)
- added J_S300: IDE, Connector_PinHeader_2.54mm:PinHeader_2x20_P2.54mm_Horizontal, F.Cu at (246.9, 224.5)
- added LS_S400: Speaker, Connector_PinHeader_2.54mm:PinHeader_1x02_P2.54mm_Vertical, F.Cu at (311.0, 236.1)
- added Q300: 2N3904, Package_TO_SOT_THT:TO-92_Inline, F.Cu at (344.1, 67.8)
- added Q_S400: NPN, Package_TO_SOT_THT:TO-92L_Inline, F.Cu at (317.9, 247.9)
- added R200: 1k, Resistor_THT:R_Axial_DIN0204_L3.6mm_D1.6mm_P5.08mm_Horizontal, F.Cu at (355.7, 180.8)
- added R201: 1k, Resistor_THT:R_Axial_DIN0204_L3.6mm_D1.6mm_P5.08mm_Horizontal, F.Cu at (355.7, 183.9)
- added R202: 1k, Resistor_THT:R_Axial_DIN0204_L3.6mm_D1.6mm_P5.08mm_Horizontal, F.Cu at (355.7, 187.1)
- added R203: 1k, Resistor_THT:R_Axial_DIN0204_L3.6mm_D1.6mm_P5.08mm_Horizontal, F.Cu at (355.7, 191.4)
- added R204: 1k, Resistor_THT:R_Axial_DIN0204_L3.6mm_D1.6mm_P5.08mm_Horizontal, F.Cu at (355.7, 194.5)
- added R205: 1k, Resistor_THT:R_Axial_DIN0204_L3.6mm_D1.6mm_P5.08mm_Horizontal, F.Cu at (355.7, 197.7)
- added R206: 1k, Resistor_THT:R_Axial_DIN0204_L3.6mm_D1.6mm_P5.08mm_Horizontal, F.Cu at (355.7, 200.8)
- added R207: 1k, Resistor_THT:R_Axial_DIN0204_L3.6mm_D1.6mm_P5.08mm_Horizontal, F.Cu at (355.7, 204.0)
- added R208: 1k, Resistor_THT:R_Axial_DIN0204_L3.6mm_D1.6mm_P5.08mm_Horizontal, F.Cu at (355.7, 207.1)
- added R209: 1k, Resistor_THT:R_Axial_DIN0204_L3.6mm_D1.6mm_P5.08mm_Horizontal, F.Cu at (355.4, 210.4)
- added R210: 1k, Resistor_THT:R_Axial_DIN0204_L3.6mm_D1.6mm_P5.08mm_Horizontal, F.Cu at (355.4, 213.6)
- added R211: 1k, Resistor_THT:R_Axial_DIN0204_L3.6mm_D1.6mm_P5.08mm_Horizontal, F.Cu at (355.4, 216.7)
- added R212: 1k, Resistor_THT:R_Axial_DIN0204_L3.6mm_D1.6mm_P5.08mm_Horizontal, F.Cu at (355.4, 226.2)
- added R213: 4k7, Resistor_THT:R_Axial_DIN0204_L3.6mm_D1.6mm_P5.08mm_Horizontal, F.Cu at (355.7, 174.5)
- added R214: 4k7, Resistor_THT:R_Axial_DIN0204_L3.6mm_D1.6mm_P5.08mm_Horizontal, F.Cu at (355.7, 177.6)
- added R300: 1k, Resistor_THT:R_Axial_DIN0204_L3.6mm_D1.6mm_P5.08mm_Horizontal, F.Cu at (352.4, 29.0)
- added R301: 1k, Resistor_THT:R_Axial_DIN0204_L3.6mm_D1.6mm_P5.08mm_Horizontal, F.Cu at (352.4, 32.1)
- added R302: 1k, Resistor_THT:R_Axial_DIN0204_L3.6mm_D1.6mm_P5.08mm_Horizontal, F.Cu at (352.4, 35.3)
- added R303: 1k, Resistor_THT:R_Axial_DIN0204_L3.6mm_D1.6mm_P5.08mm_Horizontal, F.Cu at (352.4, 38.4)
- added R304: 1k, Resistor_THT:R_Axial_DIN0204_L3.6mm_D1.6mm_P5.08mm_Horizontal, F.Cu at (352.4, 41.6)
- added R305: 1k, Resistor_THT:R_Axial_DIN0204_L3.6mm_D1.6mm_P5.08mm_Horizontal, F.Cu at (352.4, 44.7)
- added R306: 1k, Resistor_THT:R_Axial_DIN0204_L3.6mm_D1.6mm_P5.08mm_Horizontal, F.Cu at (352.4, 47.9)
- added R307: 1k, Resistor_THT:R_Axial_DIN0204_L3.6mm_D1.6mm_P5.08mm_Horizontal, F.Cu at (352.4, 51.0)
- added R308: 1k, Resistor_THT:R_Axial_DIN0204_L3.6mm_D1.6mm_P5.08mm_Horizontal, F.Cu at (360.4, 29.0)
- added R309: 1k, Resistor_THT:R_Axial_DIN0204_L3.6mm_D1.6mm_P5.08mm_Horizontal, F.Cu at (360.4, 32.1)
- added R310: 1k, Resistor_THT:R_Axial_DIN0204_L3.6mm_D1.6mm_P5.08mm_Horizontal, F.Cu at (360.4, 35.3)
- added R311: 1k, Resistor_THT:R_Axial_DIN0204_L3.6mm_D1.6mm_P5.08mm_Horizontal, F.Cu at (360.4, 38.4)
- added R312: 1k, Resistor_THT:R_Axial_DIN0204_L3.6mm_D1.6mm_P5.08mm_Horizontal, F.Cu at (360.4, 41.6)
- added R313: 330R, Resistor_THT:R_Axial_DIN0204_L3.6mm_D1.6mm_P5.08mm_Horizontal, F.Cu at (360.4, 44.7)
- added R314: 330R, Resistor_THT:R_Axial_DIN0204_L3.6mm_D1.6mm_P5.08mm_Horizontal, F.Cu at (360.4, 47.9)
- added R315: 330R, Resistor_THT:R_Axial_DIN0204_L3.6mm_D1.6mm_P5.08mm_Horizontal, F.Cu at (360.4, 51.0)
- added R316: 470R, Resistor_THT:R_Axial_DIN0204_L3.6mm_D1.6mm_P5.08mm_Horizontal, F.Cu at (343.6, 59.8)
- added R317: 1k, Resistor_THT:R_Axial_DIN0204_L3.6mm_D1.6mm_P5.08mm_Horizontal, F.Cu at (343.6, 62.9)
- added R_S300: 1k, Resistor_THT:R_Axial_DIN0204_L3.6mm_D1.6mm_P5.08mm_Horizontal, F.Cu at (255.8, 176.3)
- added R_S400: 47R, Resistor_THT:R_Axial_DIN0204_L3.6mm_D1.6mm_P5.08mm_Horizontal, F.Cu at (355.4, 223.0)
- added R_S401: 1K, Resistor_THT:R_Axial_DIN0204_L3.6mm_D1.6mm_P5.08mm_Horizontal, F.Cu at (355.4, 219.9)
- added U100: GAL16V8, Package_DIP:DIP-20_W7.62mm, F.Cu at (142.7, 203.0)
- added U101: RAM_LOW, Package_DIP:DIP-32_W15.24mm, F.Cu at (61.2, 141.2)
- added U102: RAM_HIGH, Package_DIP:DIP-32_W15.24mm, F.Cu at (81.5, 141.4)
- added U103: RAM_LOW, Package_DIP:DIP-32_W15.24mm, F.Cu at (101.9, 141.4)
- added U104: RAM_HIGH, Package_DIP:DIP-32_W15.24mm, F.Cu at (122.3, 141.5)
- added U105: RAM_LOW, Package_DIP:DIP-32_W15.24mm, F.Cu at (61.3, 188.4)
- added U106: RAM_HIGH, Package_DIP:DIP-32_W15.24mm, F.Cu at (81.6, 188.4)
- added U107: RAM_LOW, Package_DIP:DIP-32_W15.24mm, F.Cu at (101.7, 188.4)
- added U108: RAM_HIGH, Package_DIP:DIP-32_W15.24mm, F.Cu at (122.1, 188.0)
- added U200: GAL16V8, Package_DIP:DIP-20_W7.62mm, F.Cu at (264.0, 176.0)
- added U300: ~, Package_DIP:DIP-40_W15.24mm, F.Cu at (324.5, 42.1)
- added U301: 74HC245, Package_DIP:DIP-20_W7.62mm, F.Cu at (311.6, 39.4)
- added U302: 74HC245, Package_DIP:DIP-20_W7.62mm, F.Cu at (311.9, 68.1)
- added U303: 24LC256, Package_DIP:DIP-8_W7.62mm, F.Cu at (331.8, 105.2)
- added U304: GAL16V8, Package_DIP:DIP-20_W7.62mm, F.Cu at (357.1, 102.7)
- added U_S100: 82C55A, Package_DIP:DIP-40_W15.24mm, F.Cu at (364.8, 145.8)
- added U_S200: Multio, Package_DIP:DIP-40_W15.24mm, F.Cu at (319.2, 167.5)
- added U_S201: 74HC245, Package_DIP:DIP-20_W7.62mm, F.Cu at (341.2, 167.3)
- added U_S202: 74HC245, Package_DIP:DIP-20_W7.62mm, F.Cu at (341.7, 195.0)
- moved C_U10 47.5 mm to (126.2, 58.1)
- moved C_U4 47.5 mm to (121.6, 103.9)
- moved C2 47.5 mm to (39.1, 39.9)
- moved C_U13 47.5 mm to (58.3, 83.5)
- moved C_U2 47.5 mm to (149.0, 56.4)
- moved D1 47.5 mm to (41.1, 46.2)
- moved R1 47.5 mm to (90.3, 49.2)
- moved R10 47.5 mm to (44.3, 38.2)
- moved R7 47.5 mm to (48.8, 30.3)
- moved C3 47.5 mm to (90.1, 20.1)
- moved C_U0_1 47.5 mm to (90.7, 31.3)
- moved C_U0_2 47.5 mm to (132.2, 39.3)
- moved C_U1 47.5 mm to (148.8, 25.1)
- moved C_U11 47.5 mm to (74.5, 61.4)
- moved C_U12 47.5 mm to (67.9, 21.9)
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Connections:
- U3 pad 19: /Orion68-CPU-2//cpu_bus_enable -> /Orion68-CPU-2//bus_enable
- U4 pad 19: /Orion68-CPU-2//cpu_bus_enable -> /Orion68-CPU-2//bus_enable
- U5 pad 19: /Orion68-CPU-2//cpu_bus_enable -> /Orion68-CPU-2//bus_enable
- U6 pad 1: GND -> /Orion68-CPU-2//AS
- U6 pad 19: /Orion68-CPU-2//cpu_bus_enable -> /Orion68-CPU-2//bus_enable
- U8 pad 12: unconnected-(U8-IO8-Pad12) -> /Orion68-CPU-2//bus_enable
