File: schematics/Orion68/_autosave-orion68mem.kicad_sch (KiCad schematic)
At the start: 14 parts, among them J100 Euro96pin, J7 JMP_PIN3, J8 JMP_PIN31, J9 JMP_PIN29, U100 GAL20V8, U101 RAM_LOW, U102 RAM_HIGH, U103 RAM_LOW, U104 RAM_HIGH, U105 RAM_LOW, U106 RAM_HIGH, U107 RAM_LOW, U108 RAM_HIGH

Commit message: Updating...
Parts:
- J7: value JMP_PIN3 -> JMP_PIN03
- U18: value ~ -> AT29C512
Other:
- moved on the sheet: U18
Changed lines of the file:
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@@
 	(wire
 		(pts
-			(xy 58.42 -15.24) (xy 53.34 -15.24)
+			(xy 69.85 143.51) (xy 64.77 143.51)
 		)
 		(stroke
@@
 	)
 	(label "BA8"
-		(at 22.86 -31.75 180)
+		(at 34.29 127 180)
 		(effects
 			(font
@@
 	)
 	(label "BA5"
-		(at 22.86 -39.37 180)
+		(at 34.29 119.38 180)
 		(effects
 			(font
@@
 	)
 	(label "BA10"
-		(at 22.86 -26.67 180)
+		(at 34.29 132.08 180)
 		(effects
 			(font
@@
 	)
 	(label "BA12"
-		(at 22.86 -21.59 180)
+		(at 34.29 137.16 180)
 		(effects
 			(font
@@
 	)
 	(label "BA6"
-		(at 22.86 -36.83 180)
+		(at 34.29 121.92 180)
 		(effects
 			(font
@@
 	)
 	(label "BA3"
-		(at 22.86 -44.45 180)
+		(at 34.29 114.3 180)
 		(effects
 			(font
@@
 	)
 	(label "{slash}RAM1CS_L"
-		(at 53.34 -7.62 0)
+		(at 64.77 151.13 0)
 		(effects
 			(font
@@
 	)
 	(label "BA9"
-		(at 22.86 -29.21 180)
+		(at 34.29 129.54 180)
 		(effects
 			(font
@@
 	)
 	(label "B{slash}cpurd"
-		(at 53.34 -11.43 0)
+		(at 64.77 147.32 0)
 		(effects
 			(font
@@
 	)
 	(label "BA14"
-		(at 22.86 -16.51 180)
+		(at 34.29 142.24 180)
 		(effects
 			(font
@@
 	)
 	(label "BA13"
-		(at 22.86 -19.05 180)
+		(at 34.29 139.7 180)
 		(effects
 			(font
@@
 	)
 	(label "BA11"
-		(at 22.86 -24.13 180)
+		(at 34.29 134.62 180)
 		(effects
 			(font
@@
 	)
 	(label "BA2"
-		(at 22.86 -46.99 180)
+		(at 34.29 111.76 180)
 		(effects
 			(font
@@
 	)
 	(label "BA15"
-		(at 22.86 -13.97 180)
+		(at 34.29 144.78 180)
 		(effects
 			(font
@@
 	)
 	(label "BA7"
-		(at 22.86 -34.29 180)
+		(at 34.29 124.46 180)
 		(effects
 			(font
@@
 	)
 	(label "BA4"
-		(at 22.86 -41.91 180)
+		(at 34.29 116.84 180)
 		(effects
 			(font
@@
 	)
 	(label "BA16"
-		(at 22.86 -11.43 180)
+		(at 34.29 147.32 180)
 		(effects
 			(font
@@
 	)
 	(label "BA1"
-		(at 22.86 -49.53 180)
+		(at 34.29 109.22 180)
 		(effects
 			(font
@@
 	(symbol
 		(lib_id "power:+5V")
-		(at 58.42 -15.24 0)
+		(at 69.85 143.51 0)
 		(unit 1)
 		(exclude_from_sim no)
@@
 		(fields_autoplaced yes)
 		(property "Reference" "#PWR0124"
-			(at 58.42 -11.43 0)
+			(at 69.85 147.32 0)
 			(effects
 				(font
@@
 		)
 		(property "Value" "+5V"
-			(at 58.42 -20.32 0)
+			(at 69.85 138.43 0)
 			(effects
 				(font
@@
 		)
 		(property "Footprint" ""
-			(at 58.42 -15.24 0)
+			(at 69.85 143.51 0)
 			(effects
 				(font
@@
 		)
 		(property "Datasheet" ""
-			(at 58.42 -15.24 0)
+			(at 69.85 143.51 0)
 			(effects
 				(font
@@
 		)
 		(property "Description" "Power symbol creates a global label with name \"+5V\""
-			(at 58.42 -15.24 0)
+			(at 69.85 143.51 0)
 			(effects
 				(font
@@
 			)
 		)
-		(property "Value" "JMP_PIN3"
+		(property "Value" "JMP_PIN03"
 			(at 24.892 17.018 0)
 			(effects
@@
 	(symbol
 		(lib_id "pdSilva:AT29C512")
-		(at 38.1 -53.34 0)
+		(at 49.53 105.41 0)
 		(unit 1)
 		(exclude_from_sim no)
@@
 		(on_board yes)
 		(dnp no)
-		(fields_autoplaced yes)
 		(property "Reference" "U18"
-			(at 26.67 -53.34 0)
+			(at 38.1 105.41 0)
 			(do_not_autoplace yes)
 			(effects
@@
 			)
 		)
-		(property "Value" "~"
-			(at 38.1 -55.88 0)
+		(property "Value" "AT29C512"
+			(at 57.404 104.14 0)
 			(effects
 				(font
@@
 		)
 		(property "Footprint" ""
-			(at 38.1 -53.34 0)
+			(at 49.53 105.41 0)
 			(effects
 				(font
@@
 		)
 		(property "Datasheet" ""
-			(at 38.1 -53.34 0)
+			(at 49.53 105.41 0)
 			(effects
 				(font
@@
 		)
 		(property "Description" ""
-			(at 38.1 -53.34 0)
+			(at 49.53 105.41 0)
 			(effects
 				(font
