File: schematics/Orion68/_autosave-orion68_serial.kicad_sch (KiCad schematic)
At the start: 32 parts, among them J700 Euro96pin, J701 RS232_1, J702 RS232_1, J703 RS232_1, U18_C? 100nf, U20 74HC138, U701 UART1, U702 UART2, U703 UART3, Y1 14.745600

Commit message: Teclado funcionando
Connections:
- net /IORD: now also J700.72
- net /IOWR: now also J700.75
Other:
- moved on the sheet: J700
