File: schematics/Orion68/orion68mem.kicad_sch (KiCad schematic)
At the start: 31 parts, among them J100 Euro96pin, J101B TI9900_8BITS, J13 J100A, J14 J100B, J15 J100C, J16 J100A, J17 J100A, J18 J100A, J20 J101A, J29 ramRom29, J3 ramRom3, J30 rom2Rom5_30, J31 ramRom31, J7 J100A, J8 J100B, J9 J100C, U100A 74HC138, U100B 74HC138, U101A RAM_LOW, U101B RAM_HIGH, U102A RAM_LOW, U102B RAM_HIGH, U103A RAM_LOW, U103B RAM_HIGH, U104A RAM_LOW, U104B RAM_HIGH, U105A RAM_LOW, U105B RAM_HIGH, U18 AT29C512, U23 CY62256-70PC, U29 28C256

Commit message: Vbug2.0 rodando 18-06-2026
Parts:
- added J19: Conn_02x05_Counter_Clockwise, symbol Connector_Generic:Conn_02x05_Counter_Clockwise
Connections:
- net +5V: now also J30.1 (Pin_1); no longer J30.3 (Pin_3)
- net BA18: now also J30.3 (Pin_3); no longer J30.1 (Pin_1)
Other:
- note added: "J29"
- note added: "J3"
- note added: "J30"
- note added: "J30 1-2 ROM256 2-3 RAM E ROM512"
- note removed: "J30 1-2 RAM 2-3 ROM256 E ROM512"
- moved on the sheet: J30, J31
Changed lines of the file:
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@@
 		)
 	)
+	(text "J29"
+		(exclude_from_sim no)
+		(at 66.802 2.794 0)
+		(effects
+			(font
+				(size 2.27 2.27)
+			)
+		)
+	)
 	(text "Memory board  -  100"
 		(exclude_from_sim no)
@@
 		)
 	)
+	(text "J3"
+		(exclude_from_sim no)
+		(at 66.802 -15.494 0)
+		(effects
+			(font
+				(size 2.27 2.27)
+			)
+		)
+	)
 	(text "J101A\n1-2 68k\n2-3 TI_8BITS\n"
 		(exclude_from_sim no)
@@
 		)
 	)
+	(text "J30"
+		(exclude_from_sim no)
+		(at 55.372 -5.842 0)
+		(effects
+			(font
+				(size 2.27 2.27)
+			)
+		)
+	)
 	(text "REVER TODOS OS NUMEROS DOS JUMPERS ESTÁ BAGUNÇADO DEVIDO A CÓPIAS"
 		(exclude_from_sim no)
@@
 		)
 	)
-	(text "J30\n1-2 RAM\n2-3 ROM256 E ROM512\n"
+	(text "J30\n1-2 ROM256\n2-3 RAM E ROM512\n"
 		(exclude_from_sim no)
-		(at 22.606 67.564 0)
+		(at 22.606 56.134 0)
 		(effects
 			(font
@@
 	(text "J31\n1-2 RAM\n2-3 ROM512\n"
 		(exclude_from_sim no)
-		(at 22.352 54.102 0)
+		(at 22.352 68.072 0)
 		(effects
 			(font
@@
 	(wire
 		(pts
-			(xy 60.96 66.04) (xy 60.96 71.12)
-		)
-		(stroke
-			(width 0)
-			(type default)
-		)
-	)
-	(wire
-		(pts
 			(xy 303.53 78.74) (xy 303.53 80.01)
 		)
@@
 	(wire
 		(pts
-			(xy 53.34 68.58) (xy 67.31 68.58)
+			(xy 53.34 57.15) (xy 67.31 57.15)
 		)
 		(stroke
@@
 	(wire
 		(pts
-			(xy 53.34 71.12) (xy 60.96 71.12)
-		)
-		(stroke
-			(width 0)
-			(type default)
-		)
-	)
-	(wire
-		(pts
 			(xy 288.29 137.16) (xy 287.02 137.16)
 		)
@@
 	(wire
 		(pts
-			(xy 53.34 57.15) (xy 58.42 57.15)
+			(xy 53.34 71.12) (xy 58.42 71.12)
 		)
 		(stroke
@@
 	(wire
 		(pts
+			(xy 53.34 54.61) (xy 62.23 54.61)
+		)
+		(stroke
+			(width 0)
+			(type default)
+		)
+	)
+	(wire
+		(pts
 			(xy 240.03 58.42) (xy 279.4 58.42)
 		)
@@
 	(wire
 		(pts
+			(xy 62.23 50.8) (xy 62.23 54.61)
+		)
+		(stroke
+			(width 0)
+			(type default)
+		)
+	)
+	(wire
+		(pts
 			(xy 290.83 177.8) (xy 287.02 177.8)
 		)
@@
 	(wire
 		(pts
-			(xy 53.34 54.61) (xy 67.31 54.61)
+			(xy 53.34 68.58) (xy 67.31 68.58)
 		)
 		(stroke
@@
 	(wire
 		(pts
-			(xy 58.42 53.34) (xy 58.42 57.15)
+			(xy 58.42 67.31) (xy 58.42 71.12)
 		)
 		(stroke
@@
 	)
 	(label "PIN31"
-		(at 67.31 54.61 0)
+		(at 67.31 68.58 0)
 		(effects
 			(font
@@
 	)
 	(label "PIN30"
-		(at 67.31 68.58 0)
+		(at 67.31 57.15 0)
 		(effects
 			(font
@@
 	)
 	(label "BA18"
-		(at 53.34 66.04 0)
+		(at 53.34 59.69 0)
 		(effects
 			(font
@@
 	)
 	(label "A16"
-		(at 53.34 52.07 0)
+		(at 53.34 66.04 0)
 		(effects
 			(font
@@
 	(symbol
 		(lib_id "power:+5V")
-		(at 60.96 66.04 0)
+		(at 62.23 50.8 0)
 		(unit 1)
 		(exclude_from_sim no)
@@
 		(fields_autoplaced yes)
 		(property "Reference" "#PWR0111"
-			(at 60.96 69.85 0)
+			(at 62.23 54.61 0)
 			(effects
 				(font
@@
 		)
 		(property "Value" "+5V"
-			(at 60.96 60.96 0)
+			(at 62.23 45.72 0)
 			(effects
 				(font
@@
 		)
 		(property "Footprint" ""
-			(at 60.96 66.04 0)
+			(at 62.23 50.8 0)
 			(effects
 				(font
@@
 		)
 		(property "Datasheet" ""
-			(at 60.96 66.04 0)
+			(at 62.23 50.8 0)
 			(effects
 				(font
@@
 		)
 		(property "Description" "Power symbol creates a global label with name \"+5V\""
-			(at 60.96 66.04 0)
+			(at 62.23 50.8 0)
 			(effects
 				(font
@@
 	(symbol
 		(lib_id "Connector_Generic:Conn_01x03")
-		(at 48.26 68.58 0)
+		(at 48.26 57.15 0)
 		(mirror y)
 		(unit 1)
@@
 		(dnp no)
 		(property "Reference" "J30"
-			(at 51.054 60.706 0)
+			(at 51.054 49.276 0)
 			(effects
 				(font
@@
 		)
 		(property "Value" "rom2Rom5_30"
-			(at 58.166 62.738 0)
+			(at 58.166 51.308 0)
 			(effects
 				(font
@@
 		)
 		(property "Footprint" ""
-			(at 48.26 68.58 0)
+			(at 48.26 57.15 0)
 			(effects
 				(font
@@
 		)
 		(property "Datasheet" "~"
-			(at 48.26 68.58 0)
+			(at 48.26 57.15 0)
 			(effects
 				(font
@@
 		)
 		(property "Description" "Generic connector, single row, 01x03, script generated (kicad-library-utils/schlib/autogen/connector/)"
-			(at 48.26 68.58 0)
+			(at 48.26 57.15 0)
 			(effects
 				(font
@@
 	(symbol
 		(lib_id "power:+5V")
-		(at 58.42 53.34 0)
+		(at 58.42 67.31 0)
 		(mirror y)
 		(unit 1)
@@
 		(fields_autoplaced yes)
 		(property "Reference" "#PWR061"
-			(at 58.42 57.15 0)
+			(at 58.42 71.12 0)
 			(effects
 				(font
@@
 		)
 		(property "Value" "+5V"
-			(at 58.42 48.26 0)
+			(at 58.42 62.23 0)
 			(effects
 				(font
@@
 		)
 		(property "Footprint" ""
-			(at 58.42 53.34 0)
+			(at 58.42 67.31 0)
 			(effects
 				(font
@@
 		)
 		(property "Datasheet" ""
-			(at 58.42 53.34 0)
+			(at 58.42 67.31 0)
 			(effects
 				(font
@@
 		)
 		(property "Description" "Power symbol creates a global label with name \"+5V\""
-			(at 58.42 53.34 0)
+			(at 58.42 67.31 0)
 			(effects
 				(font
@@
 	(symbol
 		(lib_id "Connector_Generic:Conn_01x03")
-		(at 48.26 54.61 0)
+		(at 48.26 68.58 0)
 		(mirror y)
 		(unit 1)
@@
 		(dnp no)
 		(property "Reference" "J31"
-			(at 46.736 54.61 0)
+			(at 46.736 68.58 0)
 			(effects
 				(font
@@
 		)
 		(property "Value" "ramRom31"
-			(at 52.578 49.276 0)
+			(at 52.578 63.246 0)
 			(effects
 				(font
@@
 		)
 		(property "Footprint" ""
-			(at 48.26 54.61 0)
+			(at 48.26 68.58 0)
 			(effects
 				(font
@@
 		)
 		(property "Datasheet" "~"
-			(at 48.26 54.61 0)
+			(at 48.26 68.58 0)
 			(effects
 				(font
@@
 		)
 		(property "Description" "Generic connector, single row, 01x03, script generated (kicad-library-utils/schlib/autogen/connector/)"
-			(at 48.26 54.61 0)
+			(at 48.26 68.58 0)
 			(effects
 				(font
@@
 					(unit 1)
 				)
+			)
+		)
+	)
+	(symbol
+		(lib_id "Connector_Generic:Conn_02x05_Counter_Clockwise")
+		(at 64.77 -5.08 90)
+		(unit 1)
+		(exclude_from_sim no)
+		(in_bom yes)
+		(on_board yes)
+		(dnp no)
+		(fields_autoplaced yes)
+		(property "Reference" "J19"
+			(at 72.39 -7.6201 90)
+			(effects
+				(font
+					(size 1.27 1.27)
+				)
+				(justify right)
+				(hide yes)
+			)
+		)
+		(property "Value" "Conn_02x05_Counter_Clockwise"
+			(at 72.39 -6.3501 90)
+			(effects
+				(font
+					(size 1.27 1.27)
+				)
+				(justify right)
+				(hide yes)
+			)
+		)
+		(property "Footprint" ""
+			(at 64.77 -5.08 0)
+			(effects
+				(font
+					(size 1.27 1.27)
+				)
+				(hide yes)
+			)
+		)
+		(property "Datasheet" "~"
+			(at 64.77 -5.08 0)
+			(effects
+				(font
+					(size 1.27 1.27)
+				)
+				(hide yes)
+			)
+		)
+		(property "Description" "Generic connector, double row, 02x05, counter clockwise pin numbering scheme (similar to DIP package numbering), script generated (kicad-library-utils/schlib/autogen/connector/)"
+			(at 64.77 -5.08 0)
+			(effects
+				(font
+					(size 1.27 1.27)
+				)
+				(hide yes)
+			)
+		)
+		(pin "7"
+		)
+		(pin "5"
+		)
+		(pin "6"
+		)
+		(pin "2"
+		)
+		(pin "1"
+		)
+		(pin "3"
+		)
+		(pin "4"
+		)
+		(pin "8"
+		)
+		(pin "10"
+		)
+		(pin "9"
+		)
+		(instances
+			(project "Orion68"
+				(path "/c7ab032b-c937-44de-ab42-c91dee57f0a8/70b7defe-43f8-4fe6-9382-ae901438ae75"
+					(reference "J19")
+					(unit 1)
+				)
