File: schematics/Orion68/Orion68.kicad_sch (KiCad schematic)
At the start: 0 parts

Commit message: Orion68 OS compiled but not tested
Other:
- sheet Ide renamed rtc
Changed lines of the file:
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@@
 			(color 0 0 0 0.0000)
 		)
-		(property "Sheetname" "Ide"
+		(property "Sheetname" "rtc"
 			(at 19.304 102.6664 0)
 			(effects
