File: schematics/Orion68/ide.kicad_sch (KiCad schematic)
At the start: 29 parts, among them J4 IDE-40W, J5 PWR

Commit message: Orion68 OS compiled but not tested
Parts:
- removed C1: 100pF, symbol Device:C
- removed D6: LED, symbol Device:LED
- removed J4: IDE-40W, symbol Connector_Generic:Conn_02x20_Odd_Even
- removed J5: PWR, symbol Connector_Generic:Conn_02x01
- removed R17, R18: 2k2, symbol Device:R
- removed R600, R601, R602, R603, R604, R605, R606, R607, R608, R609, R610, R611, R612, R613, R614, R615, R616, R617, R618, R619, R620, R621, R622: 33R, symbol Device:R
Connections:
- no-connect marks 6 -> 0
