File: schematics/Orion68/cpu2.kicad_sch (KiCad schematic)
At the start: 40 parts, among them J10 Conn_02x08_Counter_Clockwise, J6 systemTickFreq, J600 Euro96pin, J601 clock, J602 clock1, Q7 2N3904, Q8 2N3904, SW3 Reset, U16 74LS139, U2.? ICM7555xB, U21 74LS20, U22 74HC164, U24 74HC4078, U600 68000D, U601 74LS393, U602 74HC74, U603 74HC14, U604 ATmega8-16P

Commit message: update
Connections:
- net BA1 is gone; now on net A1: J600.19
- net BA10 is gone; now on net A10: J600.28
- net BA11 is gone; now on net A11: J600.29
- net BA12 is gone; now on net A12: J600.30
- net BA13 is gone; now on net A13: J600.31
- net BA14 is gone; now on net A14: J600.91
- net BA15 is gone; now on net A15: J600.90
- net BA16 is gone; now on net A16: J600.89
- net BA17 is gone; now on net A17: J600.88
- net BA18 is gone; now on net A18: J600.87
- net BA19 is gone; now on net A19: J600.86
- net BA2 is gone; now on net A2: J600.20
- net BA20 is gone; now on net A20: J600.81
- net BA21 is gone; now on net A21: J600.80
- net BA22 is gone; now on net A22: J600.79
- net BA23 is gone; now on net A23: J600.78
- net BA3 is gone; now on net A3: J600.21
- net BA4 is gone; now on net A4: J600.22
- net BA5 is gone; now on net A5: J600.23
- net BA6 is gone; now on net A6: J600.24
- net BA7 is gone; now on net A7: J600.25
- net BA8 is gone; now on net A8: J600.26
- net BA9 is gone; now on net A9: J600.27
- net BD0 is gone; now on net D0: J600.2
- net BD1 is gone; now on net D1: J600.3
- net BD10 is gone; now on net D10: J600.12
- net BD11 is gone; now on net D11: J600.13
- net BD12 is gone; now on net D12: J600.14
- net BD13 is gone; now on net D13: J600.15
- net BD14 is gone; now on net D14: J600.16
- net BD15 is gone; now on net D15: J600.17
- net BD2 is gone; now on net D2: J600.4
- net BD3 is gone; now on net D3: J600.5
- net BD4 is gone; now on net D4: J600.6
- net BD5 is gone; now on net D5: J600.7
- net BD6 is gone; now on net D6: J600.8
- net BD7 is gone; now on net D7: J600.9
- net BD8 is gone; now on net D8: J600.10
- net BD9 is gone; now on net D9: J600.11
- net B/AS is gone; now on net /AS: J600.69
- net B/LDS is gone; now on net /LDS: J600.70
- net B/UDS is gone; now on net /UDS: J600.71
- net IRQ6 is gone; now on net IRQ7: J600.68
- net +12V: now also J600.95; no longer J600.92
- net GND: no longer J600.93, J600.95
- net IRQ1: now also J600.93
- net IRQ3: now also J600.76
- net IRQ4: now also J600.77
- net IRQ5: now also J600.83
