File: schematics/Orion68/orion68_serial.kicad_sch (KiCad schematic)
At the start: 65 parts, among them J11 IDE-40W, J12 PWR, J700 Euro96pin, J701 RS232_1, J702 RS232_1, J703 RS232_1, U17 74LS139, U18_C? 100nf, U19 74LS139, U20 74HC138, U701 UART1, U702 UART2, U703 UART3, Y1 14.745600

Commit message: update
Connections:
- net BA10 is gone; now on net A10: J700.28
- net BA11 is gone; now on net A11: J700.29
- net BA12 is gone; now on net A12: J700.30
- net BA13 is gone; now on net A13: J700.31
- net BA14 is gone; now on net A14: J700.91
- net BA15 is gone; now on net A15: J700.90
- net BA8 is gone; now on net A8: J700.26
- net BA9 is gone; now on net A9: J700.27
- net B/AS is gone; now on net /AS: J700.69
- net +12V: now also J700.95; no longer J700.92
- net A1: now also J700.19
- net A2: now also J700.20
- net A3: now also J700.21
- net BA1: no longer J700.19
- net BA2: no longer J700.20
- net BA3: no longer J700.21
- net BD0: no longer J700.2
- net BD1: no longer J700.3
- net BD2: no longer J700.4
- net BD3: no longer J700.5
- net BD4: no longer J700.6
- net BD5: no longer J700.7
- net BD6: no longer J700.8
- net BD7: no longer J700.9
- net GND: no longer J700.93, J700.95
- net IRQ4: now also J700.77; no longer U700.49 (IRQC)
- net IRQ5: now also J700.83, U700.21 (IRQB); no longer U700.55 (IRQD)
- net IRQ6: now also J700.92; no longer J700.68, U700.21 (IRQB)
- net /IORD: no longer J700.72
- net /IOWR: no longer J700.75
- net IRQ3: now reaches J700.76
- net BA16 renamed A16
- net BA17 renamed A17
- net BA18 renamed A18
- net BA19 renamed A19
- net BA20 renamed A20
- net BA21 renamed A21
- net BA22 renamed A22
- net BA23 renamed A23
- net BA4 renamed A4
- net BA5 renamed A5
- net BA6 renamed A6
- net BA7 renamed A7
- net BD10 renamed D10
- net BD11 renamed D11
- net BD12 renamed D12
- net BD13 renamed D13
- net BD14 renamed D14
- net BD15 renamed D15
- net BD8 renamed D8
- net BD9 renamed D9
- net B/LDS renamed /LDS
- net B/UDS renamed /UDS
- net IRQ2: no longer names the net of U700.15 (IRQA)
- new net D0: J700.2
- new net D1: J700.3
- new net D2: J700.4
- new net D3: J700.5
- new net D4: J700.6
- new net D5: J700.7
- new net D6: J700.8
- new net D7: J700.9
- new net IRQ1: J700.93
- new net IRQ7: J700.68
- new net /iord: J700.72
- new net /iowr: J700.75
