File: schematics/Orion68/orion68io.kicad_sch (KiCad schematic)
At the start: 32 parts, among them J200 Euro96pin, U200 GAL16V8

Commit message: update
Connections:
- net M/IO is gone; now on net IRQ3: J200.76
- net /BERR is gone; now on net IRQ7: J200.68
- net /SSO is gone; now on net IRQ4: J200.77
- net +12V: now also J200.95; no longer J200.92
- net BA1: no longer J200.19
- net BA10: no longer J200.28
- net BA11: no longer J200.29
- net BA2: no longer J200.20
- net BA3: no longer J200.21
- net BA4: no longer J200.22
- net BA5: no longer J200.23
- net BD0: no longer J200.2
- net BD1: no longer J200.3
- net BD10: no longer J200.12
- net BD11: no longer J200.13
- net BD12: no longer J200.14
- net BD13: no longer J200.15
- net BD14: no longer J200.16
- net BD15: no longer J200.17
- net BD2: no longer J200.4
- net BD3: no longer J200.5
- net BD4: no longer J200.6
- net BD5: no longer J200.7
- net BD6: no longer J200.8
- net BD7: no longer J200.9
- net BD8: no longer J200.10
- net BD9: no longer J200.11
- net B/cpurd: no longer J200.45
- net D0: now also J200.2
- net D1: now also J200.3
- net D2: now also J200.4
- net D3: now also J200.5
- net D4: now also J200.6
- net D5: now also J200.7
- net D6: now also J200.8
- net D7: now also J200.9
- net GND: no longer J200.93, J200.95
- net IRQ3: no longer J200.49
- net IRQ4: no longer J200.50
- net IRQ5: now also J200.83; no longer J200.89
- net IRQ7: no longer J200.91
- net TICK_IN: no longer J200.86
- net /IO_CS: now also J200.84; no longer J200.85
- net /IO_CS1: now reaches J200.82
- net ALE renamed /memrd
- net BA0: no longer names the net of J200.18
- net BA12 renamed A12
- net BA13 renamed A13
- net BA14: no longer names the net of J200.63
- net BA15: no longer names the net of J200.62
- net BA16: no longer names the net of J200.61
- net BA17: no longer names the net of J200.60
- net BA18: no longer names the net of J200.59
- net BA19: no longer names the net of J200.58
- net BA20: no longer names the net of J200.57
- net BA21: no longer names the net of J200.56
- net BA22: no longer names the net of J200.55
- net BA23: no longer names the net of J200.54
- net BA6 renamed A6
- net BA7 renamed A7
- net BA8 renamed A8
- net BA9 renamed A9
- net BOOTIN renamed A18
- net B/AS: no longer names the net of J200.43
- net B/LDS renamed /LDS
- net B/UDS renamed /UDS
- net B/cpuwr: no longer names the net of J200.46
- net CPU_CLK renamed A20
- net CRUCLK: no longer names the net of J200.35
- net CRUIN: no longer names the net of J200.36
- net CRUOUT: no longer names the net of J200.37
- net DBIN: no longer names the net of J200.38
- net DT/R renamed /iowr
- net E: no longer names the net of J200.34
- net HLDA: no longer names the net of J200.52
- net IAQ: no longer names the net of J200.39
- net IC3: no longer names the net of J200.47
- net IRQ2: no longer names the net of J200.48
- net IRQ6 renamed A15
- net NMI: no longer names the net of J200.41
- net PWR_GOOD renamed A17
- net RDY: no longer names the net of J200.44
- net Res9 renamed /AS
- net /DEN renamed /memwr
- net /HALT: no longer names the net of J200.53
- net /HOLD: no longer names the net of J200.42
- net /INTA renamed /iord
- net /INTR: no longer names the net of J200.40
- net /M1 renamed A22
- net /RFSH renamed A21
- net /RST: no longer names the net of J200.51
- net /WAIT renamed A23
- new net A1: J200.19
- new net A10: J200.28
- new net A11: J200.29
- new net A14: J200.91
- new net A16: J200.89
- new net A19: J200.86
- new net A2: J200.20
- new net A3: J200.21
- new net A4: J200.22
- new net A5: J200.23
- new net D10: J200.12
- new net D11: J200.13
- new net D12: J200.14
- new net D13: J200.15
- new net D14: J200.16
- new net D15: J200.17
- new net D8: J200.10
- new net D9: J200.11
- new net IRQ1: J200.93
- new net /MEM_CS: J200.85
Other:
- note added: "1 2 3 4 5 6 7 8 9 10 11 12 13 14 15"
- note added: "15 14 13 12 11 10 9 8 7 6 5 4 3 2 1"
