File: schematics/Orion68/orion68vid.kicad_sch (KiCad schematic)
At the start: 27 parts, among them J300 Euro96pin, Q4 2N7000, U301 74HC245, U302 74HC245, U303 24LC256, U304 GAL16V8, U305 74LS541

Commit message: update
Connections:
- net BA10 is gone; now on net A10: J300.28
- net BA11 is gone; now on net A11: J300.29
- net BA12 is gone; now on net A12: J300.30
- net BA13 is gone; now on net A13: J300.31
- net BA14 is gone; now on net A14: J300.91
- net +12V: now also J300.95; no longer J300.92
- net BA1: no longer J300.19
- net BA15: no longer J300.90
- net BA2: no longer J300.20
- net BA3: no longer J300.21
- net BA4: no longer J300.22
- net BA5: no longer J300.23
- net BD0: no longer J300.2
- net BD1: no longer J300.3
- net BD2: no longer J300.4
- net BD3: no longer J300.5
- net BD4: no longer J300.6
- net BD5: no longer J300.7
- net BD6: no longer J300.8
- net BD7: no longer J300.9
- net B/AS: no longer J300.69
- net D0: now also J300.2
- net D1: now also J300.3
- net D2: now also J300.4
- net D3: now also J300.5
- net D4: now also J300.6
- net D5: now also J300.7
- net D6: now also J300.8
- net D7: now also J300.9
- net GND: no longer J300.93, J300.95
- net /iord: now also J300.72
- net /iowr: now also J300.75
- net /memrd: now also J300.73
- net /memwr: now also J300.74
- net IRQ7: now reaches J300.68
- net IRQ3: now reaches J300.76
- net IRQ4: now reaches J300.77
- net IRQ5: now reaches J300.83
- net BA16 renamed A16
- net BA17 renamed A17
- net BA18 renamed A18
- net BA19 renamed A19
- net BA20 renamed A20
- net BA21 renamed A21
- net BA22 renamed A22
- net BA23 renamed A23
- net BA6 renamed A6
- net BA7 renamed A7
- net BA8 renamed A8
- net BA9 renamed A9
- net BD10 renamed D10
- net BD11 renamed D11
- net BD12 renamed D12
- net BD13 renamed D13
- net BD14 renamed D14
- net BD15 renamed D15
- net BD8 renamed D8
- net BD9 renamed D9
- net B/LDS renamed /LDS
- net B/UDS renamed /UDS
- new net A1: J300.19
- new net A15: J300.90
- new net A2: J300.20
- new net A3: J300.21
- new net A4: J300.22
- new net A5: J300.23
- new net IRQ1: J300.93
- new net /AS: J300.69

Commit message: RTC rcp5c01A working...
Parts:
- added J_S1: DB25_Socket, Connector_PinHeader_2.54mm:PinHeader_2x13_P2.54mm_Vertical, symbol Connector:DB25_Socket
- added U_S1: 82C55A, Package_DIP:DIP-40_W15.24mm, symbol Interface:82C55A
Connections:
- net +5V: now also U_S1.26 (VCC)
- net BA1: now also U_S1.9 (A0)
- net BA2: now also U_S1.8 (A1)
- net BD0: now also U_S1.34 (D0)
- net BD1: now also U_S1.33 (D1)
- net BD2: now also U_S1.32 (D2)
- net BD3: now also U_S1.31 (D3)
- net BD4: now also U_S1.30 (D4)
- net BD5: now also U_S1.29 (D5)
- net BD6: now also U_S1.28 (D6)
- net BD7: now also U_S1.27 (D7)
- net D0: now also J_S1.2, U_S1.4 (PA0)
- net D1: now also J_S1.3, U_S1.3 (PA1)
- net D2: now also J_S1.4, U_S1.2 (PA2)
- net D3: now also J_S1.5, U_S1.1 (PA3)
- net D4: now also J_S1.6, U_S1.40 (PA4)
- net D5: now also J_S1.7, U_S1.39 (PA5)
- net D6: now also J_S1.8, U_S1.38 (PA6)
- net D7: now also J_S1.9, U_S1.37 (PA7)
- net GND: now also J_S1.18 (P18), J_S1.19 (P19), J_S1.20 (P20), J_S1.21 (P21), J_S1.22 (P22), J_S1.23 (P23), J_S1.24 (P24), J_S1.25 (P25), U_S1.7 (GND)
- net RESET: now also U_S1.35 (RESET)
- new net BUSY: J_S1.11, U_S1.15 (PC1)
- new net B/cpurd: U_S1.5 (~{RD})
- new net B/cpurw: U_S1.36 (~{WR})
- new net CS_82C55: U_S1.6 (~{CS})
- new net STROBE: J_S1.1, U_S1.14 (PC0)
Other:
- note added: ";FF8000 !Y1 = !AS * !IOWR * !IOCS * !IOCS1 * A15 * !A14 * !A13 * !A12 * !A11 * !A10 * !A09 * !A08 ;FF9000 !Y2 = !IOWR * !IOCS * !IOCS1 * A15 * !A14 * !A13 * A12 * !A11 * !A10 * !A09 * !A08 ;FFA000 !Y3 = !IOWR * !IOCS * !IOCS1 * A15 * !A14 * A13 * !A12 * !A11 * !A10 * !A09 * !A08 ;FFB000 !Y4 = !IOWR * !IOCS * !IOCS1 * A15 * !A14 * A13 * A12 * !A11 * !A10 * !A09 * !A08"
- note added: "DB25 fêmea +-------+--------------+--------------+---------------------------------------------+ |Pino |,Nome |,Direção (PC) |,Função | +-------+--------------+--------------+---------------------------------------------+ |1 |,Strobe |,Saída |,Indica que os dados são válidos (Ativo em 0)| |2 |,D0 |,E/S |,Bit de Dados 0 (LSB) | |3 |,D1 |,E/S |,Bit de Dados 1 | |4 |,D2 |,E/S |,Bit de Dados 2 | |5 |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"
- note added: "Setor S100"
- note removed: "19 18 17 16 | 15 1 0 0 0 | 0 = F80000 1 0 0 0 | 1 = F88000 1 0 0 1 | 0 = F90000 1 0 0 1 | 1 = F98000 1 0 1 0 | 0 = FA0000 1 0 1 0 | 1 = FA8000 1 0 1 1 | 0 = FB0000 1 0 1 1 | 1 = FB8000 pino 1 (A0) = A15 do 68000 pino 2 (A1) = A16 do 68000 pino 3 (A2) = A17 do 68000 pino 4 (/E0) = A18 do 68000 pino 5 (/E1) = /LDS R/W /AS do 68000 pino 6 (E2) = A19 do 68000 com isso a saida pino 7 /Y7 só deve ser a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"
