File: hardware/schematics/Orion68/cpu2.kicad_sch (KiCad schematic)
At the start: 40 parts, among them J10 Conn_02x08_Counter_Clockwise, J6 systemTickFreq, J600 Euro96pin, J601 clock, J602 clock1, Q7 2N3904, Q8 2N3904, SW3 Reset, U16 74LS139, U2.? ICM7555xB, U21 74LS20, U22 74HC164, U24 74HC4078, U600 68000D, U601 74LS393, U602 74HC74, U603 74HC14, U604 ATmega8-16P

Commit message: New orioncor programming eeprom via ob.elf
Parts:
- removed SW3: Reset, Button_Switch_THT:SW_Push_1P2T_Vertical_E-Switch_800UDP8P1A1M6, symbol Switch:SW_Push
- removed U602: 74HC74, Package_DIP:DIP-14_W7.62mm, symbol 74xx:74HC74
- added CU601_1, CU602_1, CU603_1, CU604_1, CU605_1, CU606_1, CU607_1, CY600_1: 100nF, Capacitor_SMD:C_0805_2012Metric, symbol Device:C
- added D600: Halt, Connector_PinHeader_2.54mm:PinHeader_1x02_P2.54mm_Vertical, symbol Device:LED
- added D601: Reset, Connector_PinHeader_2.54mm:PinHeader_1x02_P2.54mm_Vertical, symbol Device:LED
- added H1, H2: MountingHole, MountingHole:MountingHole_3.2mm_M3, symbol Mechanical:MountingHole
- added H3, H4: MountingHole, MountingHole:MountingHole_2.1mm, symbol Mechanical:MountingHole
- added J602_1: clock_dtack, Connector_PinHeader_2.54mm:PinHeader_2x05_P2.54mm_Vertical, symbol Connector_Generic:Conn_02x05_Counter_Clockwise
- added J605: Conn_01x32, Connector_PinHeader_2.54mm:PinHeader_1x32_P2.54mm_Vertical, symbol Connector_Generic:Conn_01x32
- added Pin600: Clock, Connector_PinHeader_2.54mm:PinHeader_1x01_P2.54mm_Vertical, symbol Connector_Generic:Conn_01x01
- added Pin601: dtack, Connector_PinHeader_2.54mm:PinHeader_1x01_P2.54mm_Vertical, symbol Connector_Generic:Conn_01x01
- added Pin602: iord, Connector_PinHeader_2.54mm:PinHeader_1x01_P2.54mm_Vertical, symbol Connector_Generic:Conn_01x01
- added Pin603: iowr, Connector_PinHeader_2.54mm:PinHeader_1x01_P2.54mm_Vertical, symbol Connector_Generic:Conn_01x01
- added Pin604: vpa, Connector_PinHeader_2.54mm:PinHeader_1x01_P2.54mm_Vertical, symbol Connector_Generic:Conn_01x01
- added Pin605: Reset, Connector_PinHeader_2.54mm:PinHeader_1x01_P2.54mm_Vertical, symbol Connector_Generic:Conn_01x01
- added Pin606: Reset Inv., Connector_PinHeader_2.54mm:PinHeader_1x01_P2.54mm_Vertical, symbol Connector_Generic:Conn_01x01
- added Pin607: memwr, Connector_PinHeader_2.54mm:PinHeader_1x01_P2.54mm_Vertical, symbol Connector_Generic:Conn_01x01
- added Pin608: memrd, Connector_PinHeader_2.54mm:PinHeader_1x01_P2.54mm_Vertical, symbol Connector_Generic:Conn_01x01
- added Pin609: Vcc, Connector_PinHeader_2.54mm:PinHeader_1x01_P2.54mm_Vertical, symbol Connector_Generic:Conn_01x01
- added Pin610: gnd, Connector_PinHeader_2.54mm:PinHeader_1x01_P2.54mm_Vertical, symbol Connector_Generic:Conn_01x01
- added R616, R617: 470R, Resistor_THT:R_Axial_DIN0204_L3.6mm_D1.6mm_P5.08mm_Horizontal, symbol Device:R
- added SW3: Reset, Connector_PinHeader_2.54mm:PinHeader_1x02_P2.54mm_Vertical, symbol Connector_Generic:Conn_01x02
- CU600_1, CU600_2: footprint Capacitor_THT:C_Disc_D4.3mm_W1.9mm_P5.00mm -> Capacitor_SMD:C_0805_2012Metric
- D602: renamed from D?; footprint Diode_THT:D_DO-34_SOD68_P5.08mm_Vertical_AnodeUp -> Connector_PinHeader_2.54mm:PinHeader_1x02_P2.54mm_Vertical
- J603: renamed from J10; footprint (none) -> Connector_PinHeader_2.54mm:PinHeader_2x08_P2.54mm_Vertical
- J604: renamed from J6; footprint (none) -> Connector_PinHeader_2.54mm:PinHeader_2x03_P2.54mm_Vertical
- R600, R601, R602, R603, R604, R605, R606, R607: footprint Resistor_THT:R_Axial_DIN0204_L3.6mm_D1.6mm_P5.08mm_Horizontal -> Resistor_SMD:R_0805_2012Metric
- U600rst1: renamed from U2.?; footprint Package_SO:SOIC-8_3.9x4.9mm_P1.27mm -> Package_DIP:DIP-8_W7.62mm
- U601, U603: footprint (none) -> Package_DIP:DIP-14_W7.62mm
- U602: renamed from U22; footprint (none) -> Package_DIP:DIP-14_W7.62mm
- U605: renamed from U21; footprint (none) -> Package_DIP:DIP-14_W7.62mm
- U606: renamed from U24; footprint (none) -> Package_DIP:DIP-14_W7.62mm
- U607: renamed from U16; footprint (none) -> Package_DIP:DIP-16_W7.62mm
- gave numbers to parts that had none: 1
- renumbered C6 to C600, C7 to C601, C8 to C602, R25 to R608, R26 to R609, R29 to R611, R31 to R612, R32 to R613, R30 to R614
Connections:
- net IPL0 is gone; now on net /IPL0: U604.23 (PC0)
- net IPL1 is gone; now on net /IPL1: U604.24 (PC1)
- net IPL2 is gone; now on net /IPL2: U604.25 (PC2)
- net +5V: now also U601.14 (VCC), U603.14 (VCC), U605.14 (VCC), U606.14 (VCC), U607.16 (VCC), CU601_1.1, CU602_1.1, CU603_1.1, CU604_1.1, CU605_1.1, CU606_1.1, CU607_1.1, CY600_1.1, D600.2 (A), D601.2 (A), J605.17 (Pin_17), Pin609.1 (Pin_1)
- net 125khz: now also J602.5 (Pin_5); no longer J602.3 (Pin_3)
- net 16MHZ: now also U604.9 (PB6/XTAL1), J602_1.1 (Pin_1)
- net 1MHZ: now also J602_1.9 (Pin_9)
- net 250khz: now also J602.3 (Pin_3); no longer J602.2 (Pin_2)
- net 2MHZ: now also J602_1.7 (Pin_7)
- net 4MHZ: now also J602_1.5 (Pin_5); no longer U602.8 (CP)
- net 62,5khz: now also J602.7 (Pin_7); no longer J602.4 (Pin_4)
- net 8MHZ: now also J602_1.3 (Pin_3)
- net A10: now also J605.6 (Pin_6)
- net A11: now also J605.7 (Pin_7)
- net A12: now also J605.8 (Pin_8)
- net A13: now also J605.9 (Pin_9)
- net A14: now also J605.10 (Pin_10)
- net A15: now also J605.11 (Pin_11)
- net A16: now also J605.12 (Pin_12)
- net A17: now also J605.13 (Pin_13)
- net A18: now also J605.14 (Pin_14)
- net A19: now also J605.15 (Pin_15)
- net A20: now also J605.16 (Pin_16)
- net A21: now also J605.18 (Pin_18)
- net A22: now also J605.19 (Pin_19)
- net A23: now also J605.20 (Pin_20)
- net A5: now also J605.1 (Pin_1)
- net A6: now also J605.2 (Pin_2)
- net A7: now also J605.3 (Pin_3)
- net A8: now also J605.4 (Pin_4)
- net A9: now also J605.5 (Pin_5)
- net CPU_CLK: now also J602.2 (Pin_2), J602.4 (Pin_4), J602.6 (Pin_6), J602.8 (Pin_8), U600.15 (CLK), Pin600.1 (Pin_1)
- net D10: now also J605.27 (Pin_27)
- net D11: now also J605.26 (Pin_26)
- net D12: now also J605.25 (Pin_25)
- net D13: now also J605.24 (Pin_24)
- net D14: now also J605.23 (Pin_23)
- net D15: now also J605.22 (Pin_22)
- net D5: now also J605.32 (Pin_32)
- net D6: now also J605.31 (Pin_31)
- net D7: now also J605.30 (Pin_30)
- net D8: now also J605.29 (Pin_29)
- net D9: now also J605.28 (Pin_28)
- net FC0: now also U600.28 (FC0)
- net FC1: now also U600.27 (FC1)
- net FC2: now also U600.26 (FC2)
- net GND: now also J604.2 (Pin_2), U601.7 (GND), U603.7 (GND), U605.7 (GND), U606.10 (I6), U606.11 (I7), U606.12 (I8), U606.5 (I4), U606.7 (VCC), U606.9 (I5), U607.8 (GND), CU601_1.2, CU602_1.2, CU603_1.2, CU604_1.2, CU605_1.2, CU606_1.2, CU607_1.2, CY600_1.2, J605.21 (Pin_21), Pin610.1 (Pin_1), SW3.1 (Pin_1); no longer J604.5 (Pin_5)
- net IRQ2: now also U604.15 (PB1)
- net IRQ7: no longer U604.15 (PB1)
- net RESET: now also Pin606.1 (Pin_1)
- net R/W: now also Pin608.1 (Pin_1)
- net /DTACK: now also U603.8, Pin601.1 (Pin_1)
- net /HALT: now also R616.2
- net /RESET: now also Pin605.1 (Pin_1), R617.2
- net /VPA: now also Pin604.1 (Pin_1)
- net /iord: now also Pin602.1 (Pin_1)
- net /iowr: now also Pin603.1 (Pin_1)
- net /memrd: now also Pin607.1 (Pin_1)
- net at U604.27 (PC4): now also J604.3 (Pin_3); no longer J604.2 (Pin_2)
- net at U604.28 (PC5): now also J604.5 (Pin_5); no longer J604.3 (Pin_3)
- net at C600.1, R608.2, U600rst1.2 (TR): now also SW3.2 (Pin_2)
- net at J603.10 (Pin_10), J603.12 (Pin_12), J603.14 (Pin_14)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: now also J603.2 (Pin_2), J603.4 (Pin_4), J603.6 (Pin_6), J603.8 (Pin_8); no longer J603.11 (Pin_11), J603.13 (Pin_13), J603.15 (Pin_15), J603.9 (Pin_9)
- net at U602.4 (Q1): now also J603.3 (Pin_3); no longer J603.2 (Pin_2)
- net at U602.5 (Q2): now also J603.5 (Pin_5); no longer J603.3 (Pin_3)
- net at U602.6 (Q3): now also J603.7 (Pin_7); no longer J603.4 (Pin_4)
- net at U602.10 (Q4): now also J603.9 (Pin_9); no longer J603.5 (Pin_5)
- net at U602.11 (Q5): now also J603.11 (Pin_11); no longer J603.6 (Pin_6)
- net at U602.12 (Q6): now also J603.13 (Pin_13); no longer J603.7 (Pin_7)
- net at U602.13 (Q7): now also J603.15 (Pin_15); no longer J603.8 (Pin_8)
- net /CS_MULTIO: no longer names the net of J600.60
- net /DTACK_AUTO: no longer names the net of J600.62
- net /DTACK_AUTO: no longer U603.8
- net /DTACK_CPU: no longer names the net of J600.63
- net /DTACK_MIO: no longer names the net of J600.61
- net /DTACK_PVGA: no longer names the net of J600.59
- new net: J602_1.10 (Pin_10), J602_1.2 (Pin_2), J602_1.4 (Pin_4), J602_1.6 (Pin_6), J602_1.8 (Pin_8), U602.8 (CP)
- new net: D600.1 (K), R616.1
- new net: D601.1 (K), R617.1
- no-connect marks 2 -> 6
Other:
- note removed: "FALTA IMPLEMENTAR"
- note removed: "NÃO IMPLEMENTADO AINDA"
- note removed: "livre"
- moved on the sheet: C600, C601, C602, CU600_1, CU600_2, D602, J601, J602, J603, J604, Q7, Q8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
