File: hardware/schematics/Orion68/orion68io.kicad_sch (KiCad schematic)
At the start: 45 parts, among them IC4 XR68C681CJTR-F, J1 LevelConverter, J200 Euro96pin, J22 Kbd_usb, J23 Conn_01x06, J26 DuartB, J28 DuartA, Q4 3.6864MHz, U200 GAL16V8, U25 SN74LVC245APW, U26 SN74LVC245APW, U30 LM2937xT, U33 68681, U36 UART2

Commit message: Code running well after clean-up
Connections:
- net /CS_MULTIO_C is gone; now on net /CS_MIO: U26.7 (A6)
- net /CS_RTC: no longer names the net of U200.17 (I03)
Changed lines of the file:
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@@
-		)
-	)
-	(label "{slash}CS_MULTIO_C"
-		(at 208.28 177.8 0)
-		(effects
-			(font
-				(size 1.27 1.27)
-			)
-			(justify left bottom)
 		)
 	)
@@
 		)
 	)
+	(label "{slash}CS_MIO"
+		(at 208.28 177.8 0)
+		(effects
+			(font
+				(size 1.27 1.27)
+			)
+			(justify left bottom)
+		)
+	)
 	(label "D0"
 		(at 369.57 21.59 0)
@@
 		)
 	)
-	(label "{slash}CS_RTC"
-		(at 55.88 254 0)
-		(effects
-			(font
-				(size 1.27 1.27)
-			)
-			(justify left bottom)
-		)
-	)

Commit message: Changing from gal16v8 to 22v10
Parts:
- added U16: 74HC138, symbol 74xx:74HC138
- added U21: 74HC4078, Package_DIP:DIP-14_W7.62mm, symbol pdSilva:74HC4078
- added U22: 74LS08, symbol 74xx:74LS08
Connections:
- net /DT_DUART is gone; now on net PRETO: U33.9 (DTACK)
- net +5V: now also U16.16 (VCC), U21.14 (VCC), U22.14 (VCC)
- net A08: now also U16.1 (A0)
- net A09: now also U16.2 (A1)
- net A10: now also U16.3 (A2)
- net A11: now also U21.2 (I1)
- net A12: now also U22.1
- net A13: now also U21.3 (I2)
- net A14: now also U21.4 (I3)
- net A15: now also U22.2
- net GND: now also U16.8 (GND), U21.11 (I7), U21.12 (I8), U21.7 (VCC), U22.7 (GND)
- net /AS: now also U21.5 (I4)
- net /CS_DUART: now also U16.15 (~{Y0})
- net /CS_MIO: now also U16.14 (~{Y1})
- net /IO_CS: now also U21.9 (I5)
- net /IO_CS1: now also U21.10 (I6)
- new net: U16.6 (E2), U22.3
- new net: U16.4 (~{E0}), U16.5 (~{E1}), U21.1 (O1)
Other:
- moved on the sheet: U200
